Commit message: add inertial macros for sphere, box, and cylinder in xacro files

File: description/robot_core.xacro (robot description, xacro)
@@ -1,4 +1,5 @@
 <?xml version="1.0"?>
 <robot xmlns:xacro="http://www.ros.org/wiki/xacro" name="my_robot">
+  <xacro:include filename="inertial_macros.xacro" />
   <!-- Definición del enlace base -->
   <link name="base_link">
@@ -11,4 +12,9 @@
       </material>
     </visual>
+    <collision>
+      <geometry>
+        <box size="0 0 0"/>
+      </geometry>
+    </collision>
   </link>
   <!-- Definición del cubo simple -->
@@ -19,4 +25,12 @@
       </geometry>
     </visual>
+    <collision>
+      <geometry>
+        <box size="0.5 0.5 0.25"/>
+      </geometry>
+    </collision>
+    <xacro:inertial_box mass="0.5" x="0.5" y= "0.5" z="0.25">
+      <origin xyz="0 0 0" rpy="0 0 0"/>
+    </xacro:inertial_box>
   </link>
   <!-- Definición de la articulación del cubo -->
@@ -36,4 +50,9 @@
       </material>
     </visual>
+    <collision>
+      <geometry>
+        <cylinder radius="0.0" length="0.0"/>
+      </geometry>
+    </collision>
   </link>
   <!-- Articulación para conectar cylinder_link a base_link -->
@@ -59,4 +78,12 @@
       </material>
     </visual>
+    <collision>
+      <geometry>
+        <cylinder radius="0.1" length="0.05"/>
+      </geometry>
+    </collision>
+    <xacro:inertial_cylinder mass="0.1" radius="0.1" length="0.05">
+      <origin xyz="0 0 0" rpy="0 0 0"/>
+    </xacro:inertial_cylinder>
   </link>
   <!-- Definición de la articulación de la rueda izquierda -->
@@ -76,4 +103,12 @@
       </material>
     </visual>
+    <collision>
+      <geometry>
+        <cylinder radius="0.1" length="0.05"/>
+      </geometry>
+    </collision>
+    <xacro:inertial_cylinder mass="0.1" radius="0.1" length="0.05">
+      <origin xyz="0 0 0" rpy="0 0 0"/>
+    </xacro:inertial_cylinder>
   </link>
   <!-- Definición de la esfera -->
@@ -87,4 +122,12 @@
       </material>
     </visual>
+    <collision>
+      <geometry>
+        <sphere radius="0.1"/>
+      </geometry>
+    </collision>
+    <xacro:inertial_sphere mass="0.1" radius="0.1">
+      <origin xyz="0 0 0" rpy="0 0 0"/>
+    </xacro:inertial_sphere>
   </link>
   <!-- Articulación para conectar sphere_link a base_link -->

Commit message: add Gazebo materials for robot links and create launch file for simulation

File: description/robot_core.xacro (robot description, xacro)
@@ -18,4 +18,7 @@
     </collision>
   </link>
+  <gazebo reference="base_link">
+    <material>Gazebo/Grey</material>
+  </gazebo>
   <!-- Definición del cubo simple -->
   <link name="cube_link">
@@ -34,4 +37,7 @@
     </xacro:inertial_box>
   </link>
+  <gazebo reference="cube_link">
+    <material>Gazebo/Color</material>
+  </gazebo>
   <!-- Definición de la articulación del cubo -->
   <joint name="cube_joint" type="fixed">
@@ -56,4 +62,7 @@
     </collision>
   </link>
+  <gazebo reference="cylinder_link">
+    <material>Gazebo/Blue</material>
+  </gazebo>
   <!-- Articulación para conectar cylinder_link a base_link -->
   <joint name="cylinder_joint" type="fixed">
@@ -87,4 +96,7 @@
     </xacro:inertial_cylinder>
   </link>
+  <gazebo reference="right_wheel_link">
+    <material>Gazebo/Blue</material>
+  </gazebo>
   <!-- Definición de la articulación de la rueda izquierda -->
   <joint name="left_wheel_joint" type="fixed">
@@ -112,4 +124,7 @@
     </xacro:inertial_cylinder>
   </link>
+  <gazebo reference="left_wheel_link">
+    <material>Gazebo/Blue</material>
+  </gazebo>
   <!-- Definición de la esfera -->
   <link name="sphere_link">
@@ -131,4 +146,7 @@
     </xacro:inertial_sphere>
   </link>
+  <gazebo reference="sphere_link">
+    <material>Gazebo/Black</material>
+  </gazebo>
   <!-- Articulación para conectar sphere_link a base_link -->
   <joint name="sphere_joint" type="fixed">

Commit message: add gazebo control plugin and RViz configuration for robot visualization

File: description/robot_core.xacro (robot description, xacro)
@@ -1,157 +1,125 @@
 <?xml version="1.0"?>
-<robot xmlns:xacro="http://www.ros.org/wiki/xacro" name="my_robot">
-  <xacro:include filename="inertial_macros.xacro" />
-  <!-- Definición del enlace base -->
-  <link name="base_link">
-    <visual>
-      <geometry>
-        <box size="0 0 0"/> <!-- Tamaño del enlace base -->
-      </geometry>
-      <material name="grey">
-        <color rgba="0.5 0.5 0.5 1"/>
-      </material>
-    </visual>
-    <collision>
-      <geometry>
-        <box size="0 0 0"/>
-      </geometry>
-    </collision>
-  </link>
-  <gazebo reference="base_link">
-    <material>Gazebo/Grey</material>
-  </gazebo>
-  <!-- Definición del cubo simple -->
-  <link name="cube_link">
-    <visual>
-      <geometry>
-        <box size="0.5 0.5 0.25"/>
-      </geometry>
-    </visual>
-    <collision>
-      <geometry>
-        <box size="0.5 0.5 0.25"/>
-      </geometry>
-    </collision>
-    <xacro:inertial_box mass="0.5" x="0.5" y= "0.5" z="0.25">
-      <origin xyz="0 0 0" rpy="0 0 0"/>
-    </xacro:inertial_box>
-  </link>
-  <gazebo reference="cube_link">
-    <material>Gazebo/Color</material>
-  </gazebo>
-  <!-- Definición de la articulación del cubo -->
-  <joint name="cube_joint" type="fixed">
-    <parent link="base_link"/>
-    <child link="cube_link"/>
-    <origin xyz="0.1 0 0.2" rpy="0 0 0"/>
-  </joint>
-  <!-- Definicion de cilindro 1-->
-  <link name="cylinder_link">
-    <visual>
-      <geometry>
-          <cylinder radius="0.0" length="0.0"/>
-      </geometry>
-      <material name="blue">
-        <color rgba="0 0 1 1"/>
-      </material>
-    </visual>
-    <collision>
-      <geometry>
-        <cylinder radius="0.0" length="0.0"/>
-      </geometry>
-    </collision>
-  </link>
-  <gazebo reference="cylinder_link">
-    <material>Gazebo/Blue</material>
-  </gazebo>
-  <!-- Articulación para conectar cylinder_link a base_link -->
-  <joint name="cylinder_joint" type="fixed">
-    <parent link="base_link"/>
-    <child link="cylinder_link"/>
-    <origin xyz="0 0 0.1" rpy="0 0 0"/>
-  </joint>
-  <!-- Definición de la articulación de la rueda derecha -->
-  <joint name="right_wheel_joint" type="fixed">
-    <parent link="base_link"/>
-    <child link="right_wheel_link"/>
-    <origin xyz="0 0.275 0.1" rpy="-${pi/2} 0 0"/>
-  </joint>
-  <!-- Definición de la rueda derecha -->
-  <link name="right_wheel_link">
-    <visual>
-      <geometry>
-          <cylinder radius="0.1" length="0.05"/>
-      </geometry>
-      <material name="blue">
-        <color rgba="0 0 1 1"/>
-      </material>
-    </visual>
-    <collision>
-      <geometry>
-        <cylinder radius="0.1" length="0.05"/>
-      </geometry>
-    </collision>
-    <xacro:inertial_cylinder mass="0.1" radius="0.1" length="0.05">
-      <origin xyz="0 0 0" rpy="0 0 0"/>
-    </xacro:inertial_cylinder>
-  </link>
-  <gazebo reference="right_wheel_link">
-    <material>Gazebo/Blue</material>
-  </gazebo>
-  <!-- Definición de la articulación de la rueda izquierda -->
-  <joint name="left_wheel_joint" type="fixed">
-    <parent link="base_link"/>
-    <child link="left_wheel_link"/>
-    <origin xyz="0 -0.275 0.1" rpy="${-pi/2} 0 0"/>
-  </joint>
-  <!-- Definición de la rueda izquierda -->
-  <link name="left_wheel_link">
-    <visual>
-      <geometry>
-          <cylinder radius="0.1" length="0.05"/>
-      </geometry>
-      <material name="blue">
-        <color rgba="0 0 1 1"/>
-      </material>
-    </visual>
-    <collision>
-      <geometry>
-        <cylinder radius="0.1" length="0.05"/>
-      </geometry>
-    </collision>
-    <xacro:inertial_cylinder mass="0.1" radius="0.1" length="0.05">
-      <origin xyz="0 0 0" rpy="0 0 0"/>
-    </xacro:inertial_cylinder>
-  </link>
-  <gazebo reference="left_wheel_link">
-    <material>Gazebo/Blue</material>
-  </gazebo>
-  <!-- Definición de la esfera -->
-  <link name="sphere_link">
-    <visual>
-      <geometry>
-        <sphere radius="0.1"/>
-      </geometry>
-      <material name="black">
+<robot xmlns:xacro="http://www.ros.org/wiki/xacro" >
+    <xacro:include filename="inertial_macros.xacro"/>
+    <material name="white">
+        <color rgba="1 1 1 1" />
+    </material>
+    <material name="orange">
+        <color rgba="1 0.3 0.1 1"/>
+    </material>
+    <material name="blue">
+        <color rgba="0.2 0.2 1 1"/>
+    </material>
+    <material name="black">
         <color rgba="0 0 0 1"/>
-      </material>
-    </visual>
-    <collision>
-      <geometry>
-        <sphere radius="0.1"/>
-      </geometry>
-    </collision>
-    <xacro:inertial_sphere mass="0.1" radius="0.1">
-      <origin xyz="0 0 0" rpy="0 0 0"/>
-    </xacro:inertial_sphere>
-  </link>
-  <gazebo reference="sphere_link">
-    <material>Gazebo/Black</material>
-  </gazebo>
-  <!-- Articulación para conectar sphere_link a base_link -->
-  <joint name="sphere_joint" type="fixed">
-    <parent link="base_link"/>
-    <child link="sphere_link"/>
-    <origin xyz="0.25 0 0.1" rpy="0 0 0"/>
-  </joint>
+    </material>
+    <!-- BASE LINK -->
+    <link name="base_link">
+    </link>
+    <!-- CHASSIS LINK -->
+    <joint name="chassis_joint" type="fixed">
+        <parent link="base_link"/>
+        <child link="chassis"/>
+        <origin xyz="-0.1 0 0"/>
+    </joint>
+    <link name="chassis">
+        <visual>
+            <origin xyz="0.15 0 0.075"/>
+            <geometry>
+                <box size="0.3 0.3 0.15"/>
+            </geometry>
+            <material name="white"/>
+        </visual>
+        <collision>
+            <origin xyz="0.15 0 0.075"/>
+            <geometry>
+                <box size="0.3 0.3 0.15"/>
+            </geometry>
+        </collision>
+        <xacro:inertial_box mass="0.5" x="0.3" y="0.3" z="0.15">
+            <origin xyz="0.15 0 0.075" rpy="0 0 0"/>
+        </xacro:inertial_box>
+    </link>
+    <gazebo reference="chassis">
+        <material>Gazebo/White</material>
+    </gazebo>
+    <!-- LEFT WHEEL LINK -->
+    <joint name="left_wheel_joint" type="continuous">
+        <parent link="base_link"/>
+        <child link="left_wheel"/>
+        <origin xyz="0 0.175 0" rpy="-${pi/2} 0 0" />
+        <axis xyz="0 0 1"/>
+    </joint>
+    <link name="left_wheel">
+        <visual>
+            <geometry>
+                <cylinder radius="0.05" length="0.04"/>
+            </geometry>
+            <material name="blue"/>
+        </visual>
+        <collision>
+            <geometry>
+                <cylinder radius="0.05" length="0.04"/>
+            </geometry>
+        </collision>
+        <xacro:inertial_cylinder mass="0.1" length="0.04" radius="0.05">
+            <origin xyz="0 0 0" rpy="0 0 0"/>
+        </xacro:inertial_cylinder>
+    </link>
+    <gazebo reference="left_wheel">
+        <material>Gazebo/Blue</material>
+    </gazebo>
+    <!-- RIGHT WHEEL LINK -->
+    <joint name="right_wheel_joint" type="continuous">
+        <parent link="base_link"/>
+        <child link="right_wheel"/>
+        <origin xyz="0 -0.175 0" rpy="${pi/2} 0 0" />
+        <axis xyz="0 0 -1"/>
+    </joint>
+    <link name="right_wheel">
+        <visual>
+            <geometry>
+                <cylinder radius="0.05" length="0.04"/>
+            </geometry>
+            <material name="blue"/>
+        </visual>
+        <collision>
+            <geometry>
+                <cylinder radius="0.05" length="0.04"/>
+            </geometry>
+        </collision>
+        <xacro:inertial_cylinder mass="0.1" length="0.04" radius="0.05">
+            <origin xyz="0 0 0" rpy="0 0 0"/>
+        </xacro:inertial_cylinder>
+    </link>
+    <gazebo reference="right_wheel">
+        <material>Gazebo/Blue</material>
+    </gazebo>
+    <!-- CASTER WHEEL LINK -->
+    <joint name="caster_wheel_joint" type="fixed">
+        <parent link="chassis"/>
+        <child link="caster_wheel"/>
+        <origin xyz="0.24 0 0"/>
+    </joint>
+    <link name="caster_wheel">
+        <visual>
+            <geometry>
+                <sphere radius="0.05"/>
+            </geometry>
+            <material name="black"/>
+        </visual>
+        <collision>
+            <geometry>
+                <sphere radius="0.05"/>
+            </geometry>
+        </collision>
+        <xacro:inertial_sphere mass="0.1" radius="0.05">
+            <origin xyz="0 0 0" rpy="0 0 0"/>
+        </xacro:inertial_sphere>
+    </link>
+    <gazebo reference="caster_wheel">
+        <material>Gazebo/Black</material>
+        <mu1 value="0.001"/>
+        <mu2 value="0.001"/>
+    </gazebo>
 </robot>
